File: stepper.kicad_sch (KiCad schematic)
At the start: 67 parts, among them J201 M0_OUT, J202 M2_OUT, J203 M1_OUT, J204 M3_OUT, J205 M0_DIAG, J206 M1_DIAG, J207 M2_DIAG, J208 M3_DIAG, J209 M0_STOP, J210 M1_STOP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

Commit message: Auto-commit Fri Feb 17 13:50:17 EST 2023
Parts:
- U201, U202, U203, U204: footprint Package_DFN_QFN:QFN-28-1EP_5x5mm_P0.5mm_EP3.75x3.75mm_ThermalVias -> Package_DFN_QFN:QFN-28-1EP_5x5mm_P0.5mm_EP3.75x3.75mm
Changed lines of the file:
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@@
     (pin "1")
   )
-  (symbol (lib_id "matei:TMC2209") (at 67.31 52.07 0) (unit 1)
+  (symbol (lib_name "TMC2209_3") (lib_id "matei:TMC2209") (at 67.31 52.07 0) (unit 1)
     (in_bom yes) (on_board yes)
     (property "Reference" "U201" (id 0) (at 63.5 50.8 0)
@@
       (effects (font (size 1.27 1.27)) (justify left))
     )
-    (property "Footprint" "Package_DFN_QFN:QFN-28-1EP_5x5mm_P0.5mm_EP3.75x3.75mm_ThermalVias" (id 2) (at 68.58 92.71 0)
+    (property "Footprint" "Package_DFN_QFN:QFN-28-1EP_5x5mm_P0.5mm_EP3.75x3.75mm" (id 2) (at 68.58 92.71 0)
       (effects (font (size 1.27 1.27)) hide)
     )
@@
     (pin "2")
   )
-  (symbol (lib_id "matei:TMC2209") (at 65.405 137.16 0) (unit 1)
+  (symbol (lib_name "TMC2209_2") (lib_id "matei:TMC2209") (at 65.405 137.16 0) (unit 1)
     (in_bom yes) (on_board yes)
     (property "Reference" "U202" (id 0) (at 61.595 135.89 0)
@@
       (effects (font (size 1.27 1.27)) (justify left))
     )
-    (property "Footprint" "Package_DFN_QFN:QFN-28-1EP_5x5mm_P0.5mm_EP3.75x3.75mm_ThermalVias" (id 2) (at 66.675 177.8 0)
+    (property "Footprint" "Package_DFN_QFN:QFN-28-1EP_5x5mm_P0.5mm_EP3.75x3.75mm" (id 2) (at 66.675 177.8 0)
       (effects (font (size 1.27 1.27)) hide)
     )
@@
       (effects (font (size 1.27 1.27)) (justify left))
     )
-    (property "Footprint" "Package_DFN_QFN:QFN-28-1EP_5x5mm_P0.5mm_EP3.75x3.75mm_ThermalVias" (id 2) (at 158.75 92.71 0)
+    (property "Footprint" "Package_DFN_QFN:QFN-28-1EP_5x5mm_P0.5mm_EP3.75x3.75mm" (id 2) (at 158.75 92.71 0)
       (effects (font (size 1.27 1.27)) hide)
     )
@@
     (pin "2")
   )
-  (symbol (lib_id "matei:TMC2209") (at 155.575 137.16 0) (unit 1)
+  (symbol (lib_name "TMC2209_1") (lib_id "matei:TMC2209") (at 155.575 137.16 0) (unit 1)
     (in_bom yes) (on_board yes)
     (property "Reference" "U204" (id 0) (at 151.765 135.89 0)
@@
       (effects (font (size 1.27 1.27)) (justify left))
     )
-    (property "Footprint" "Package_DFN_QFN:QFN-28-1EP_5x5mm_P0.5mm_EP3.75x3.75mm_ThermalVias" (id 2) (at 156.845 177.8 0)
-      (effects (font (size 1.27 1.27)) hide)
-    )
+    (property "Footprint" "Package_DFN_QFN:QFN-28-1EP_5x5mm_P0.5mm_EP3.75x3.75mm" (id 2) (at 156.845 177.8 0)
+      (effects (font (size 1.27 1.27)) hide)
+    )
